File: Hardware/Instrument/instrument.kicad_sch (KiCad schematic)
At the start: 13 parts, among them J1 Esp32 socket, J3 Esp32 socket, SW1 SW_SPST, U2 MCP6002-xP

Commit message: Updated PDF.
Other:
- note removed: "LP filter?"
- moved on the sheet: C5, U2B, U2C
Changed lines of the file:
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@@
     (company "Studentorchesteret den Ohmske Motstanden")
   )
-  (junction (at 53.34 147.32) (diameter 0) (color 0 0 0 0)
+  (junction (at 59.69 139.7) (diameter 0) (color 0 0 0 0)
   )
   (junction (at 80.01 87.63) (diameter 0) (color 0 0 0 0)
@@
   (junction (at 62.23 90.17) (diameter 0) (color 0 0 0 0)
   )
-  (junction (at 53.34 127) (diameter 0) (color 0 0 0 0)
+  (junction (at 59.69 119.38) (diameter 0) (color 0 0 0 0)
   )
   (junction (at 62.23 95.25) (diameter 0) (color 0 0 0 0)
   )
-  (no_connect (at 63.5 137.16))
+  (no_connect (at 69.85 129.54))
   (wire (pts (xy 59.69 90.17) (xy 62.23 90.17))
     (stroke (width 0) (type default))
@@
     (stroke (width 0) (type default))
   )
-  (wire (pts (xy 53.34 149.86) (xy 53.34 147.32))
+  (wire (pts (xy 59.69 142.24) (xy 59.69 139.7))
     (stroke (width 0) (type default))
   )
@@
     (stroke (width 0) (type default))
   )
-  (wire (pts (xy 53.34 124.46) (xy 53.34 127))
+  (wire (pts (xy 59.69 116.84) (xy 59.69 119.38))
     (stroke (width 0) (type default))
   )
@@
     (stroke (width 0) (type default))
   )
-  (wire (pts (xy 53.34 127) (xy 43.18 127))
+  (wire (pts (xy 59.69 119.38) (xy 49.53 119.38))
     (stroke (width 0) (type default))
   )
@@
     (stroke (width 0) (type default))
   )
-  (wire (pts (xy 53.34 127) (xy 53.34 129.54))
+  (wire (pts (xy 59.69 119.38) (xy 59.69 121.92))
     (stroke (width 0) (type default))
   )
@@
     (stroke (width 0) (type default))
   )
-  (wire (pts (xy 53.34 147.32) (xy 53.34 144.78))
+  (wire (pts (xy 59.69 139.7) (xy 59.69 137.16))
     (stroke (width 0) (type default))
   )
@@
     (stroke (width 0) (type default))
   )
-  (wire (pts (xy 43.18 127) (xy 43.18 134.62))
+  (wire (pts (xy 49.53 119.38) (xy 49.53 127))
     (stroke (width 0) (type default))
   )
@@
     (stroke (width 0) (type default))
   )
-  (wire (pts (xy 48.26 134.62) (xy 48.26 139.7))
+  (wire (pts (xy 54.61 127) (xy 54.61 132.08))
     (stroke (width 0) (type default))
   )
@@
     (stroke (width 0) (type default))
   )
-  (wire (pts (xy 43.18 147.32) (xy 53.34 147.32))
+  (wire (pts (xy 49.53 139.7) (xy 59.69 139.7))
     (stroke (width 0) (type default))
   )
@@
     (stroke (width 0) (type default))
   )
-  (wire (pts (xy 43.18 139.7) (xy 43.18 147.32))
+  (wire (pts (xy 49.53 132.08) (xy 49.53 139.7))
     (stroke (width 0) (type default))
   )
@@
     )
   )
-  (text "LP filter?" (at 86.36 87.63 0)
-    (effects (font (size 1.27 1.27)) (justify left bottom))
-  )
   (text "ESP32\n" (at 107.95 78.74 0)
     (effects (font (size 5 5)) (justify left bottom))
@@
     (effects (font (size 1.27 1.27)) (justify left bottom))
   )
-  (symbol (lib_id "Device:C_Small") (at 43.18 137.16 180) (unit 1)
+  (symbol (lib_id "Device:C_Small") (at 49.53 129.54 180) (unit 1)
     (in_bom yes) (on_board yes) (dnp no)
-    (property "Reference" "C5" (at 37.465 135.255 90)
+    (property "Reference" "C5" (at 43.815 127.635 90)
       (effects (font (size 1.27 1.27)))
     )
-    (property "Value" "100nF" (at 40.005 135.255 90)
+    (property "Value" "100nF" (at 46.355 127.635 90)
       (effects (font (size 1.27 1.27)))
     )
-    (property "Footprint" "" (at 43.18 137.16 0)
+    (property "Footprint" "" (at 49.53 129.54 0)
       (effects (font (size 1.27 1.27)) hide)
     )
-    (property "Datasheet" "~" (at 43.18 137.16 0)
+    (property "Datasheet" "~" (at 49.53 129.54 0)
       (effects (font (size 1.27 1.27)) hide)
     )
@@
     )
   )
-  (symbol (lib_id "power:+3.3V") (at 53.34 124.46 0) (unit 1)
+  (symbol (lib_id "power:+3.3V") (at 59.69 116.84 0) (unit 1)
     (in_bom yes) (on_board yes) (dnp no) (fields_autoplaced)
-    (property "Reference" "#PWR03" (at 53.34 128.27 0)
+    (property "Reference" "#PWR03" (at 59.69 120.65 0)
       (effects (font (size 1.27 1.27)) hide)
     )
-    (property "Value" "+3.3V" (at 53.34 119.38 0)
+    (property "Value" "+3.3V" (at 59.69 111.76 0)
       (effects (font (size 1.27 1.27)))
     )
-    (property "Footprint" "" (at 53.34 124.46 0)
+    (property "Footprint" "" (at 59.69 116.84 0)
       (effects (font (size 1.27 1.27)) hide)
     )
-    (property "Datasheet" "" (at 53.34 124.46 0)
+    (property "Datasheet" "" (at 59.69 116.84 0)
       (effects (font (size 1.27 1.27)) hide)
     )
@@
     )
   )
-  (symbol (lib_id "Amplifier_Operational:MCP6002-xP") (at 55.88 137.16 0) (unit 3)
+  (symbol (lib_id "Amplifier_Operational:MCP6002-xP") (at 62.23 129.54 0) (unit 3)
     (in_bom yes) (on_board yes) (dnp no)
-    (property "Reference" "U2" (at 55.88 142.24 0)
+    (property "Reference" "U2" (at 62.23 134.62 0)
       (effects (font (size 1.27 1.27)) (justify left))
     )
-    (property "Value" "MCP6002-xP" (at 55.88 144.78 0)
+    (property "Value" "MCP6002-xP" (at 62.23 137.16 0)
       (effects (font (size 1.27 1.27)) (justify left))
     )
-    (property "Footprint" "" (at 55.88 137.16 0)
+    (property "Footprint" "" (at 62.23 129.54 0)
       (effects (font (size 1.27 1.27)) hide)
     )
-    (property "Datasheet" "http://ww1.microchip.com/downloads/en/DeviceDoc/21733j.pdf" (at 55.88 137.16 0)
+    (property "Datasheet" "http://ww1.microchip.com/downloads/en/DeviceDoc/21733j.pdf" (at 62.23 129.54 0)
       (effects (font (size 1.27 1.27)) hide)
     )
@@
     )
   )
-  (symbol (lib_id "power:GND") (at 53.34 149.86 0) (unit 1)
+  (symbol (lib_id "power:GND") (at 59.69 142.24 0) (unit 1)
     (in_bom yes) (on_board yes) (dnp no)
-    (property "Reference" "#PWR02" (at 53.34 156.21 0)
+    (property "Reference" "#PWR02" (at 59.69 148.59 0)
       (effects (font (size 1.27 1.27)) hide)
     )
-    (property "Value" "GND" (at 54.61 154.94 0)
+    (property "Value" "GND" (at 60.96 147.32 0)
       (effects (font (size 1.27 1.27)))
     )
-    (property "Footprint" "" (at 53.34 149.86 0)
+    (property "Footprint" "" (at 59.69 142.24 0)
       (effects (font (size 1.27 1.27)) hide)
     )
-    (property "Datasheet" "" (at 53.34 149.86 0)
+    (property "Datasheet" "" (at 59.69 142.24 0)
       (effects (font (size 1.27 1.27)) hide)
     )
@@
     )
   )
-  (symbol (lib_id "Amplifier_Operational:MCP6002-xP") (at 55.88 137.16 0) (unit 2)
+  (symbol (lib_id "Amplifier_Operational:MCP6002-xP") (at 62.23 129.54 0) (unit 2)
     (in_bom yes) (on_board yes) (dnp no)
-    (property "Reference" "U2" (at 60.96 128.27 0)
+    (property "Reference" "U2" (at 67.31 120.65 0)
       (effects (font (size 1.27 1.27)))
     )
-    (property "Value" "MCP6002-xP" (at 60.96 130.81 0)
+    (property "Value" "MCP6002-xP" (at 67.31 123.19 0)
       (effects (font (size 1.27 1.27)))
     )
-    (property "Footprint" "" (at 55.88 137.16 0)
+    (property "Footprint" "" (at 62.23 129.54 0)
       (effects (font (size 1.27 1.27)) hide)
     )
-    (property "Datasheet" "http://ww1.microchip.com/downloads/en/DeviceDoc/21733j.pdf" (at 55.88 137.16 0)
+    (property "Datasheet" "http://ww1.microchip.com/downloads/en/DeviceDoc/21733j.pdf" (at 62.23 129.54 0)
       (effects (font (size 1.27 1.27)) hide)
     )
